File: submission.kicad_pcb (KiCad board)
At the start: 2 copper layers, 5 parts, among them U1 L7805

Commit message: uploading submission
Parts:
- added J1: Conn_01x01_Socket, Connector_PinSocket_2.00mm:PinSocket_1x01_P2.00mm_Horizontal, F.Cu at (145.9, 104.9)
- added J2: Conn_01x01_Socket, Connector_PinSocket_2.00mm:PinSocket_1x01_P2.00mm_Horizontal, F.Cu at (145.9, 109.0)
- added J3: Conn_01x01_Socket, Connector_PinSocket_2.00mm:PinSocket_1x01_P2.00mm_Horizontal, F.Cu at (145.9, 113.0)
- added J4: Conn_01x01_Socket, Connector_PinSocket_2.00mm:PinSocket_1x01_P2.00mm_Horizontal, F.Cu at (145.9, 117.0)
- C1, C2: footprint Capacitor_SMD:C_0201_0603Metric -> Capacitor_SMD:C_0805_2012Metric
- D1: footprint LED_THT:LED_D1.8mm_W1.8mm_H2.4mm_Horizontal_O6.35mm_Z8.2mm -> LED_SMD:LED_0805_2012Metric
- R1: footprint Resistor_SMD:R_0201_0603Metric -> Resistor_SMD:R_0805_2012Metric
- U1: footprint Package_TO_SOT_THT:TO-220-2_Vertical -> Package_TO_SOT_THT:TO-220-3_Vertical
- moved U1 31.8 mm to (140.4, 123.0)
- moved R1 28.5 mm to (150.1, 113.4)
- moved C2 22.7 mm to (150.1, 107.4)
- moved D1 21.4 mm to (150.1, 110.4)
- moved C1 17.2 mm to (150.1, 104.4)
Connections:
- net Net-(U1-IN) renamed 9V
- C2 pad 1: Net-(U1-OUT) -> 5V
- R1 pad 1: Net-(U1-OUT) -> 5V

Commit message: uploading submission
Parts:
- removed J1, J2, J3, J4: Conn_01x01_Socket, Connector_PinSocket_2.00mm:PinSocket_1x01_P2.00mm_Horizontal
- added 5V1: Conn_01x01_Socket, Connector_PinSocket_2.00mm:PinSocket_1x01_P2.00mm_Horizontal, F.Cu at (134.3, 84.0)
- added 5VGND1: Conn_01x01_Socket, Connector_PinSocket_2.00mm:PinSocket_1x01_P2.00mm_Horizontal, F.Cu at (133.3, 100.0)
- added 9V1: Conn_01x01_Socket, Connector_PinSocket_2.00mm:PinSocket_1x01_P2.00mm_Horizontal, F.Cu at (151.7, 84.0)
- added 9VGND1: Conn_01x01_Socket, Connector_PinSocket_2.00mm:PinSocket_1x01_P2.00mm_Horizontal, F.Cu at (151.7, 99.5)
- U1: footprint Package_TO_SOT_THT:TO-220-3_Vertical -> Package_TO_SOT_THT:TO-220-3_Horizontal_TabUp
- moved D1 31.1 mm to (128.1, 88.5)
- moved R1 28.2 mm to (127.9, 96.0)
- moved U1 23.2 mm to (145.0, 100.2), turned to 180 degrees
- moved C2 23.0 mm to (133.1, 92.0)
- moved C1 15.8 mm to (156.6, 90.0)
